File: hardware/kicad/OpenSolarNode-RevA/01B_BQ24650.kicad_sch (KiCad schematic)
At the start: 0 parts

Commit message: feat(power): reserve hardware charge-current configuration block
Other:
- note added: "0805 preferred / 0603 minimum"
- note added: "4-position DIP switch"
- note added: "CHARGE CURRENT - CONFIGURATION RESERVATION"
- note added: "DIP contacts select only the programming network - never the charge-current path"
- note added: "PROGRAMMING RESISTOR NETWORK"
- note added: "RevB: reserve architectural/PCB allowance for a future digital potentiometer; not fitted in RevA"
- note added: "SW_CHG_CURRENT"
- note added: "Silkscreen reservation: CHARGE CURRENT + mapping table (mapping TBD)"
- note added: "THT / hand-solderable"
- note added: "TP_CHG_PROGRAM: reserve test-point location; final node TBD"
- note added: "Values + truth table: TBD in HANDOFF #002"
Changed lines of the file:
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@@
+(kicad_sch
+	(version 20250114)
+	(generator "eeschema")
+	(generator_version "10.0")
+	(paper "A4")
+	(title_block (title "OpenSolarNode - 01B BQ24650") (rev "RevA") (company "OpenSolarNode") (comment 1 "License: TBD - requires project owner approval") (comment 2 "Charge-current configuration reservation - HANDOFF 001A"))
+	(rectangle (start 25.4 25.4) (end 152.4 101.6) (stroke (width 0) (type default)) (fill (type none)))
+	(rectangle (start 35.56 50.8) (end 76.2 81.28) (stroke (width 0) (type default)) (fill (type none)))
+	(rectangle (start 91.44 50.8) (end 137.16 81.28) (stroke (width 0) (type default)) (fill (type none)))
+	(text "CHARGE CURRENT - CONFIGURATION RESERVATION" (exclude_from_sim no) (at 30.48 35.56 0) (effects (font (size 1.27 1.27) (bold yes)) (justify left bottom)))
+	(text "SW_CHG_CURRENT" (exclude_from_sim no) (at 40.64 58.42 0) (effects (font (size 1.27 1.27) (bold yes)) (justify left bottom)))
+	(text "4-position DIP switch" (exclude_from_sim no) (at 40.64 66.04 0) (effects (font (size 1.27 1.27)) (justify left bottom)))
+	(text "THT / hand-solderable" (exclude_from_sim no) (at 40.64 73.66 0) (effects (font (size 1.27 1.27)) (justify left bottom)))
+	(text "PROGRAMMING RESISTOR NETWORK" (exclude_from_sim no) (at 96.52 58.42 0) (effects (font (size 1.27 1.27) (bold yes)) (justify left bottom)))
+	(text "0805 preferred / 0603 minimum" (exclude_from_sim no) (at 96.52 66.04 0) (effects (font (size 1.27 1.27)) (justify left bottom)))
+	(text "Values + truth table: TBD in HANDOFF #002" (exclude_from_sim no) (at 96.52 73.66 0) (effects (font (size 1.27 1.27)) (justify left bottom)))
+	(text "TP_CHG_PROGRAM: reserve test-point location; final node TBD" (exclude_from_sim no) (at 35.56 91.44 0) (effects (font (size 1.27 1.27)) (justify left bottom)))
+	(text "DIP contacts select only the programming network - never the charge-current path" (exclude_from_sim no) (at 30.48 111.76 0) (effects (font (size 1.27 1.27) (bold yes)) (justify left bottom)))
+	(text "RevB: reserve architectural/PCB allowance for a future digital potentiometer; not fitted in RevA" (exclude_from_sim no) (at 30.48 121.92 0) (effects (font (size 1.27 1.27)) (justify left bottom)))
+	(text "Silkscreen reservation: CHARGE CURRENT + mapping table (mapping TBD)" (exclude_from_sim no) (at 30.48 132.08 0) (effects (font (size 1.27 1.27)) (justify left bottom)))
+	(sheet_instances (path "/" (page "4")))
+	(embedded_fonts no)
+)
